File: hw/Expression Input.kicad_sch (KiCad schematic)
At the start: 10 parts, among them J6 Exp, J7 Exp Connector, U7 NE5532

Commit message: updated hardware issues for PBC revision 2
Parts:
- U7: footprint Package_SO:SOIC-8_5.3x5.3mm_P1.27mm -> NE5532DR:NE5532DR
Changed lines of the file:
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@@
 			)
 		)
-		(property "Footprint" "Package_SO:SOIC-8_5.3x5.3mm_P1.27mm"
+		(property "Footprint" "NE5532DR:NE5532DR"
 			(at 231.14 52.07 0)
 			(effects
@@
 			)
 		)
-		(property "Footprint" "Package_SO:SOIC-8_5.3x5.3mm_P1.27mm"
+		(property "Footprint" "NE5532DR:NE5532DR"
 			(at 157.48 107.95 0)
 			(effects
@@
 			)
 		)
-		(property "Footprint" "Package_SO:SOIC-8_5.3x5.3mm_P1.27mm"
+		(property "Footprint" "NE5532DR:NE5532DR"
 			(at 62.23 153.67 0)
 			(effects
