File: hw/Midi Connector.kicad_sch (KiCad schematic)
At the start: 18 parts, among them J2 Midi In, J3 Midi Out, J4 Midi Thru, U5 74HC14, U6 H11L1

Commit message: updated hardware issues for PBC revision 2
Parts:
- J2, J3, J4: footprint DIN5_MIDI:DIN5_MIDI -> DIN5_MIDI_MultiGround:DIN5_MIDI_MultiGround
Changed lines of the file:
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@@
 			)
 		)
-		(property "Footprint" "DIN5_MIDI:DIN5_MIDI"
+		(property "Footprint" "DIN5_MIDI_MultiGround:DIN5_MIDI_MultiGround"
 			(at 62.23 157.48 0)
 			(effects
@@
 			)
 		)
-		(property "Footprint" "DIN5_MIDI:DIN5_MIDI"
+		(property "Footprint" "DIN5_MIDI_MultiGround:DIN5_MIDI_MultiGround"
 			(at 62.23 76.2 0)
 			(effects
@@
 			)
 		)
-		(property "Footprint" "DIN5_MIDI:DIN5_MIDI"
+		(property "Footprint" "DIN5_MIDI_MultiGround:DIN5_MIDI_MultiGround"
 			(at 62.23 116.84 0)
 			(effects
