File: hw/Expression_Inputs.kicad_sch (KiCad schematic)
At the start: 0 parts

Commit message: updates to hardware layer
Other:
- sheet Expression Input 1 ports: added VR, VS; removed EXP_IN
- sheet Expression Input 2 ports: added VR, VS; removed EXP_IN
- sheet Expression Input 3 ports: added VR, VS; removed EXP_IN
- sheet Expression Input 4 ports: added VR, VS; removed EXP_IN
Changed lines of the file:
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@@
 	(wire
 		(pts
-			(xy 143.51 113.03) (xy 146.05 113.03)
-		)
-		(stroke
-			(width 0)
-			(type default)
-		)
-	)
-	(wire
-		(pts
-			(xy 143.51 138.43) (xy 146.05 138.43)
-		)
-		(stroke
-			(width 0)
-			(type default)
-		)
-	)
-	(wire
-		(pts
-			(xy 143.51 62.23) (xy 146.05 62.23)
-		)
-		(stroke
-			(width 0)
-			(type default)
-		)
-	)
-	(wire
-		(pts
-			(xy 143.51 87.63) (xy 146.05 87.63)
-		)
-		(stroke
-			(width 0)
-			(type default)
+			(xy 143.51 86.36) (xy 146.05 86.36)
+		)
+		(stroke
+			(width 0)
+			(type default)
+		)
+	)
+	(wire
+		(pts
+			(xy 146.05 111.76) (xy 143.51 111.76)
+		)
+		(stroke
+			(width 0)
+			(type default)
+		)
+	)
+	(wire
+		(pts
+			(xy 143.51 88.9) (xy 146.05 88.9)
+		)
+		(stroke
+			(width 0)
+			(type default)
+		)
+	)
+	(wire
+		(pts
+			(xy 143.51 60.96) (xy 146.05 60.96)
+		)
+		(stroke
+			(width 0)
+			(type default)
+		)
+	)
+	(wire
+		(pts
+			(xy 146.05 139.7) (xy 143.51 139.7)
+		)
+		(stroke
+			(width 0)
+			(type default)
+		)
+	)
+	(wire
+		(pts
+			(xy 146.05 114.3) (xy 143.51 114.3)
+		)
+		(stroke
+			(width 0)
+			(type default)
+		)
+	)
+	(wire
+		(pts
+			(xy 143.51 63.5) (xy 146.05 63.5)
+		)
+		(stroke
+			(width 0)
+			(type default)
+		)
+	)
+	(wire
+		(pts
+			(xy 146.05 137.16) (xy 143.51 137.16)
+		)
+		(stroke
+			(width 0)
+			(type default)
+		)
+	)
+	(global_label "STM_ADC2_IN17"
+		(shape input)
+		(at 146.05 111.76 0)
+		(fields_autoplaced yes)
+		(effects
+			(font
+				(size 1.27 1.27)
+			)
+			(justify left)
+		)
+		(property "Intersheetrefs" "${INTERSHEET_REFS}"
+			(at 163.7913 111.76 0)
+			(effects
+				(font
+					(size 1.27 1.27)
+				)
+				(justify left)
+				(hide yes)
+			)
 		)
 	)
 	(global_label "STM_ADC1_IN4"
 		(shape input)
-		(at 146.05 62.23 0)
-		(fields_autoplaced yes)
-		(effects
-			(font
-				(size 1.27 1.27)
-			)
-			(justify left)
-		)
-		(property "Intersheetrefs" "${INTERSHEET_REFS}"
-			(at 162.5818 62.23 0)
+		(at 146.05 88.9 0)
+		(fields_autoplaced yes)
+		(effects
+			(font
+				(size 1.27 1.27)
+			)
+			(justify left)
+		)
+		(property "Intersheetrefs" "${INTERSHEET_REFS}"
+			(at 162.5818 88.9 0)
 			(effects
 				(font
@@
 	(global_label "STM_ADC1_IN1"
 		(shape input)
-		(at 146.05 138.43 0)
-		(fields_autoplaced yes)
-		(effects
-			(font
-				(size 1.27 1.27)
-			)
-			(justify left)
-		)
-		(property "Intersheetrefs" "${INTERSHEET_REFS}"
-			(at 162.5818 138.43 0)
+		(at 146.05 60.96 0)
+		(fields_autoplaced yes)
+		(effects
+			(font
+				(size 1.27 1.27)
+			)
+			(justify left)
+		)
+		(property "Intersheetrefs" "${INTERSHEET_REFS}"
+			(at 162.5818 60.96 0)
 			(effects
 				(font
@@
 	(global_label "STM_ADC1_IN3"
 		(shape input)
-		(at 146.05 87.63 0)
-		(fields_autoplaced yes)
-		(effects
-			(font
-				(size 1.27 1.27)
-			)
-			(justify left)
-		)
-		(property "Intersheetrefs" "${INTERSHEET_REFS}"
-			(at 162.5818 87.63 0)
+		(at 146.05 86.36 0)
+		(fields_autoplaced yes)
+		(effects
+			(font
+				(size 1.27 1.27)
+			)
+			(justify left)
+		)
+		(property "Intersheetrefs" "${INTERSHEET_REFS}"
+			(at 162.5818 86.36 0)
+			(effects
+				(font
+					(size 1.27 1.27)
+				)
+				(justify left)
+				(hide yes)
+			)
+		)
+	)
+	(global_label "STM_ADC2_IN13"
+		(shape input)
+		(at 146.05 114.3 0)
+		(fields_autoplaced yes)
+		(effects
+			(font
+				(size 1.27 1.27)
+			)
+			(justify left)
+		)
+		(property "Intersheetrefs" "${INTERSHEET_REFS}"
+			(at 163.7913 114.3 0)
 			(effects
 				(font
@@
 	(global_label "STM_ADC1_IN2"
 		(shape input)
-		(at 146.05 113.03 0)
-		(fields_autoplaced yes)
-		(effects
-			(font
-				(size 1.27 1.27)
-			)
-			(justify left)
-		)
-		(property "Intersheetrefs" "${INTERSHEET_REFS}"
-			(at 162.5818 113.03 0)
+		(at 146.05 63.5 0)
+		(fields_autoplaced yes)
+		(effects
+			(font
+				(size 1.27 1.27)
+			)
+			(justify left)
+		)
+		(property "Intersheetrefs" "${INTERSHEET_REFS}"
+			(at 162.5818 63.5 0)
+			(effects
+				(font
+					(size 1.27 1.27)
+				)
+				(justify left)
+				(hide yes)
+			)
+		)
+	)
+	(global_label "STM_ADC2_IN4"
+		(shape input)
+		(at 146.05 139.7 0)
+		(fields_autoplaced yes)
+		(effects
+			(font
+				(size 1.27 1.27)
+			)
+			(justify left)
+		)
+		(property "Intersheetrefs" "${INTERSHEET_REFS}"
+			(at 162.5818 139.7 0)
+			(effects
+				(font
+					(size 1.27 1.27)
+				)
+				(justify left)
+				(hide yes)
+			)
+		)
+	)
+	(global_label "STM_ADC2_IN3"
+		(shape input)
+		(at 146.05 137.16 0)
+		(fields_autoplaced yes)
+		(effects
+			(font
+				(size 1.27 1.27)
+			)
+			(justify left)
+		)
+		(property "Intersheetrefs" "${INTERSHEET_REFS}"
+			(at 162.5818 137.16 0)
 			(effects
 				(font
@@
 			)
 		)
-		(pin "EXP_IN" input
-			(at 143.51 62.23 0)
+		(pin "VR" input
+			(at 143.51 60.96 0)
+			(effects
+				(font
+					(size 1.27 1.27)
+				)
+				(justify right)
+			)
+		)
+		(pin "VS" input
+			(at 143.51 63.5 0)
 			(effects
 				(font
@@
 			)
 		)
-		(pin "EXP_IN" input
-			(at 143.51 138.43 0)
+		(pin "VR" input
+			(at 143.51 137.16 0)
+			(effects
+				(font
+					(size 1.27 1.27)
+				)
+				(justify right)
+			)
+		)
+		(pin "VS" input
+			(at 143.51 139.7 0)
 			(effects
 				(font
@@
 			)
 		)
-		(pin "EXP_IN" input
-			(at 143.51 87.63 0)
+		(pin "VR" input
+			(at 143.51 86.36 0)
+			(effects
+				(font
+					(size 1.27 1.27)
+				)
+				(justify right)
+			)
+		)
+		(pin "VS" input
+			(at 143.51 88.9 0)
 			(effects
 				(font
@@
 			)
 		)
-		(pin "EXP_IN" input
-			(at 143.51 113.03 0)
-			(effects
-				(font
+		(pin "VR" input
+			(at 143.51 111.76 0)
+			(effects
+				(font
+					(size 1.27 1.27)
+				)
+				(justify right)
+			)
+		)
+		(pin "VS" input
+			(at 143.51 114.3 0)
+			(effects
+				(font

Commit message: fixed input range issue
Other:
- sheet Expression Input 1 ports: added VT; removed VS
- sheet Expression Input 2 ports: added VT; removed VS
- sheet Expression Input 3 ports: added VT; removed VS
- sheet Expression Input 4 ports: added VT; removed VS
Changed lines of the file:
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@@
 			)
 		)
-		(pin "VS" input
+		(pin "VT" input
 			(at 143.51 63.5 0)
 			(effects
@@
 			)
 		)
-		(pin "VS" input
+		(pin "VT" input
 			(at 143.51 139.7 0)
 			(effects
@@
 			)
 		)
-		(pin "VS" input
+		(pin "VT" input
 			(at 143.51 88.9 0)
 			(effects
@@
 			)
 		)
-		(pin "VS" input
+		(pin "VT" input
 			(at 143.51 114.3 0)
 			(effects
